File: klp_expander/klp_expander/hub.kicad_sch (KiCad schematic)
At the start: 24 parts, among them U5 USB2514B_Bi, X1 X322525MRB4SI

Commit message: feat: merge middle mcu into klp expander. both projects will be merged and will get a new name
Connections:
- net USB_P3_PWR: no longer names the net of U5.18 (PRTPWR3/BC_EN3)
- net USB_P4_PWR: no longer names the net of U5.20 (PRTPWR4/BC_EN4)
- no-connect marks 6 -> 8
Changed lines of the file:
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@@
+	)
+	(no_connect
+		(at 142.24 97.79)
 	)
 	(no_connect
@@
 	)
 	(no_connect
+		(at 142.24 110.49)
+	)
+	(no_connect
 		(at 142.24 72.39)
 	)
@@
 	(wire
 		(pts
-			(xy 142.24 97.79) (xy 147.32 97.79)
-		)
-		(stroke
-			(width 0)
-			(type default)
-		)
-	)
-	(wire
-		(pts
 			(xy 116.84 48.26) (xy 127 48.26)
 		)
@@
 		(pts
 			(xy 96.52 48.26) (xy 106.68 48.26)
-		)
-		(stroke
-			(width 0)
-			(type default)
-		)
-	)
-	(wire
-		(pts
-			(xy 142.24 110.49) (xy 147.32 110.49)
 		)
 		(stroke
@@
 		)
 	)
-	(hierarchical_label "USB_P3_PWR"
-		(shape output)
-		(at 147.32 97.79 0)
+	(hierarchical_label "IN_DP"
+		(shape bidirectional)
+		(at 72.39 74.93 180)
+		(effects
+			(font
+				(size 1.27 1.27)
+			)
+			(justify right)
+		)
+	)
+	(hierarchical_label "USB_P3_DP"
+		(shape bidirectional)
+		(at 147.32 95.25 0)
 		(effects
 			(font
@@
 		)
 	)
-	(hierarchical_label "IN_DP"
-		(shape bidirectional)
-		(at 72.39 74.93 180)
+	(hierarchical_label "IN_DN"
+		(shape bidirectional)
+		(at 72.39 72.39 180)
 		(effects
 			(font
@@
 		)
 	)
-	(hierarchical_label "USB_P3_DP"
-		(shape bidirectional)
-		(at 147.32 95.25 0)
+	(hierarchical_label "USB_P2_DN"
+		(shape bidirectional)
+		(at 147.32 80.01 0)
 		(effects
 			(font
@@
 		)
 	)
-	(hierarchical_label "IN_DN"
-		(shape bidirectional)
-		(at 72.39 72.39 180)
-		(effects
-			(font
-				(size 1.27 1.27)
-			)
-			(justify right)
-		)
-	)
-	(hierarchical_label "USB_P2_DN"
-		(shape bidirectional)
-		(at 147.32 80.01 0)
+	(hierarchical_label "USB_P2_DP"
+		(shape bidirectional)
+		(at 147.32 82.55 0)
 		(effects
 			(font
@@
 		)
 	)
-	(hierarchical_label "USB_P2_DP"
-		(shape bidirectional)
-		(at 147.32 82.55 0)
+	(hierarchical_label "USB_P4_DN"
+		(shape bidirectional)
+		(at 147.32 105.41 0)
 		(effects
 			(font
@@
 		)
 	)
-	(hierarchical_label "USB_P4_DN"
-		(shape bidirectional)
-		(at 147.32 105.41 0)
-		(effects
-			(font
-				(size 1.27 1.27)
-			)
-			(justify left)
-		)
-	)
 	(hierarchical_label "USB_P1_DP"
 		(shape bidirectional)
@@
 		(effects
 			(font
-				(size 1.27 1.27)
-			)
-			(justify left)
-		)
-	)
-	(hierarchical_label "USB_P4_PWR"
-		(shape output)
-		(at 147.32 110.49 0)
-		(effects
-			(font
