File: klp_expander/klp_expander/mcu.kicad_sch (KiCad schematic)
At the start: 32 parts, among them SW1 SW_Push, SW2 SW_Push, U1 RP2350_60QFN, U3 W25Q128JVS, Y1 ABM8-272-T3

Commit message: update schematics
Parts:
- removed R1, R9: DNF, Resistor_SMD:R_0402_1005Metric, symbol Device:R
- removed R10: 0, Resistor_SMD:R_0402_1005Metric, symbol Device:R
Connections:
- net FLASH_SS is gone; now on net QSPI_SS: U3.1 (~{CS})
- net GPIO0: no longer names the net of U1.2 (GPIO0)
- net GPIO1: no longer names the net of U1.3 (GPIO1)
- net GPIO10: no longer names the net of U1.14 (GPIO10)
- net GPIO11: no longer names the net of U1.15 (GPIO11)
- net GPIO12: no longer names the net of U1.16 (GPIO12)
- net GPIO13: no longer names the net of U1.17 (GPIO13)
- net GPIO14: no longer names the net of U1.18 (GPIO14)
- net GPIO15: no longer names the net of U1.19 (GPIO15)
- net GPIO16: no longer names the net of U1.27 (GPIO16)
- net GPIO17: no longer names the net of U1.28 (GPIO17)
- net GPIO18: no longer names the net of U1.29 (GPIO18)
- net GPIO19: no longer names the net of U1.31 (GPIO19)
- net GPIO2: no longer names the net of U1.4 (GPIO2)
- net GPIO20: no longer names the net of U1.32 (GPIO20)
- net GPIO21: no longer names the net of U1.33 (GPIO21)
- net GPIO22 renamed GPIO_22
- net GPIO23 renamed GPIO_23
- net GPIO24 renamed GPIO_24
- net GPIO25 renamed GPIO_25
- net GPIO26_ADC0 renamed GPIO_26
- net GPIO27_ADC1 renamed GPIO_27
- net GPIO28_ADC2: no longer names the net of U1.42 (GPIO28_ADC2)
- net GPIO29_ADC3: no longer names the net of U1.43 (GPIO29_ADC3)
- net GPIO3: no longer names the net of U1.5 (GPIO3)
- net GPIO4: no longer names the net of U1.7 (GPIO4)
- net GPIO5: no longer names the net of U1.8 (GPIO5)
- net GPIO6: no longer names the net of U1.9 (GPIO6)
- net GPIO7: no longer names the net of U1.10 (GPIO7)
- net GPIO8: no longer names the net of U1.12 (GPIO8)
- net GPIO9: no longer names the net of U1.13 (GPIO9)
- net USB_D+ renamed USB_P1_DP
- net USB_D- renamed USB_P1_DN

Commit message: feat: merge middle mcu into klp expander. both projects will be merged and will get a new name
Connections:
- net LED_PWM: now reaches U1.14 (GPIO10)
- net CAN_RX: now reaches U1.15 (GPIO11)
- net CAN_TX: now reaches U1.16 (GPIO12)
- net FIL_SWITCH: now reaches U1.19 (GPIO15)
- net FIL_MOTION: now reaches U1.27 (GPIO16)
- net GPIO_17: now reaches U1.28 (GPIO17)
- net GPIO_18: now reaches U1.29 (GPIO18)
- net GPIO_19: now reaches U1.31 (GPIO19)
- net GPIO_20: now reaches U1.32 (GPIO20)
- net GPIO_21: now reaches U1.33 (GPIO21)
- net TH0: now reaches U1.42 (GPIO28_ADC2)
- net TH1: now reaches U1.43 (GPIO29_ADC3)
- net GPIO_26 renamed I2C_SDA
- net GPIO_27 renamed I2C_SCL
